Commit message: FIX: Add simplify .dae to gripper colision

File: kortex_description/grippers/gen3_lite_2f/urdf/gen3_lite_2f_macro.xacro (robot description, xacro)
@@ -13,7 +13,53 @@
     use_internal_bus_gripper_comm:=true
     moveit_active:=false">
-  <xacro:if value="${use_fake_hardware or sim_isaac or sim_gazebo}">
+    <!-- ========================================== -->
+    <!-- 1. DEFINIÇÃO DE CONTEXTO E PROPRIEDADES    -->
+    <!-- ========================================== -->
+    <xacro:property name="is_sim" value="${(use_fake_hardware or sim_isaac or sim_gazebo) and not moveit_active}"/>
+    <xacro:property name="is_real" value="${not (use_fake_hardware or sim_isaac or sim_gazebo) and not moveit_active}"/>
+    <!-- Parâmetros para ambiente MoveIt -->
+    <xacro:if value="${moveit_active}">
+      <xacro:property name="pfx" value=""/>
+      <xacro:property name="prnt" value="dummy_link"/>
+      <xacro:property name="mesh_url" value="package://kortex_description/grippers/gen3_lite_2f/meshes/"/>
+      <!-- Limites das juntas no MoveIt -->
+      <xacro:property name="rfb_rpy" value="0 1.5708 0"/>
+      <xacro:property name="rfb_lower" value="0.0"/> <xacro:property name="rfb_upper" value="0.96"/>
+      <xacro:property name="rfb_eff" value="1000"/>  <xacro:property name="rfb_vel" value="0.6"/>
+      <xacro:property name="lfb_rpy" value="0 1.5708 0"/>
+      <xacro:property name="lfb_lower" value="-0.96"/> <xacro:property name="lfb_upper" value="0.0"/>
+      <xacro:property name="lfb_eff" value="1000"/>  <xacro:property name="lfb_vel" value="1000"/>
+      <xacro:property name="lfb_mimic_m" value="-1.0"/> <xacro:property name="lfb_mimic_o" value="0.0"/>
+      <xacro:property name="tip_mimic_m" value="-0.676"/> <xacro:property name="tip_mimic_o" value="0.149"/>
+    </xacro:if>
+    <!-- Parâmetros para simulação ou hardware real -->
     <xacro:unless value="${moveit_active}">
-    <!-- ros2 control include -->
+      <xacro:property name="pfx" value="${prefix}"/>
+      <xacro:property name="prnt" value="${parent}"/>
+      <xacro:property name="mesh_url" value="file://$(find kortex_description)/grippers/gen3_lite_2f/meshes/"/>
+      <xacro:property name="rfb_rpy" value="1.571 0.611 1.571"/>
+      <xacro:property name="lfb_rpy" value="-1.571 0.611 -1.571"/>
+      <xacro:property name="lfb_mimic_m" value="1.0"/> <xacro:property name="lfb_mimic_o" value="0.0"/>
+      <xacro:property name="tip_mimic_m" value="-0.276"/> <xacro:property name="tip_mimic_o" value="-0.1"/>
+      <!-- SIMULAÇÃO -->
+      <xacro:if value="${is_sim}">
+        <xacro:property name="rfb_lower" value="-0.1"/> <xacro:property name="rfb_upper" value="0.96"/>
+        <xacro:property name="rfb_eff" value="10"/>    <xacro:property name="rfb_vel" value="0.6"/>
+        <xacro:property name="lfb_lower" value="-0.1"/> <xacro:property name="lfb_upper" value="0.96"/>
+        <xacro:property name="lfb_eff" value="10"/>    <xacro:property name="lfb_vel" value="0.6"/>
+      </xacro:if>
+      <!-- HARDWARE REAL -->
+      <xacro:if value="${is_real}">
+        <!-- TODO(MarqRazz) look into why the joint and limits needed to be flipped and modified -->
+        <xacro:property name="rfb_lower" value="0.0"/>  <xacro:property name="rfb_upper" value="0.85"/>
+        <xacro:property name="rfb_eff" value="50"/>     <xacro:property name="rfb_vel" value="0.6"/>
+        <xacro:property name="lfb_lower" value="0.0"/>  <xacro:property name="lfb_upper" value="0.85"/>
+        <xacro:property name="lfb_eff" value="1000"/>   <xacro:property name="lfb_vel" value="1000"/>
+      </xacro:if>
+    </xacro:unless>
+    <!-- ========================================== -->
+    <!-- 2. ROS2 CONTROL (APENAS SIMULAÇÃO)         -->
+    <!-- ========================================== -->
+    <xacro:if value="${is_sim}">
       <xacro:include filename="$(find kortex_description)/grippers/gen3_lite_2f/urdf/gen3_lite_2f.ros2_control.xacro" />
       <xacro:if value="${sim_gazebo}">
@@ -27,53 +73,51 @@
       </xacro:unless>
       <xacro:gripper_ros2_control
-        prefix="${prefix}"
-        use_fake_hardware="${use_fake_hardware}"
-        fake_sensor_commands="${fake_sensor_commands}"
-        sim_gazebo="${sim_gazebo}"
-        sim_isaac="${sim_isaac}"
-        isaac_joint_commands="${isaac_joint_commands}"
-        isaac_joint_states="${isaac_joint_states}"
-        tf_prefix=""/>
-  <!-- Tool frame used by the arm -->
-      <link name="${prefix}tool_frame"/>
-      <joint name="${prefix}tool_frame_joint" type="fixed">
-          <origin xyz="0 0 0.130" rpy="0 0 1.57079632679" />
-          <parent link="${parent}" />
-          <child link="${prefix}tool_frame" />
-          <axis xyz="0 0 0" />
-      </joint>
-      <!-- Gripper description -->
-      <joint name="${prefix}gripper_base_joint" type="fixed">
+        prefix="${prefix}" use_fake_hardware="${use_fake_hardware}" fake_sensor_commands="${fake_sensor_commands}"
+        sim_gazebo="${sim_gazebo}" sim_isaac="${sim_isaac}" isaac_joint_commands="${isaac_joint_commands}"
+        isaac_joint_states="${isaac_joint_states}" tf_prefix=""/>
+    </xacro:if>
+    <!-- ========================================== -->
+    <!-- 3. MACRO DE GEOMETRIA (DRY)                -->
+    <!-- ========================================== -->
+    <xacro:macro name="gripper_mesh" params="mesh_name color_rgba">
+      <visual>
         <origin xyz="0 0 0" rpy="0 0 0" />
-        <parent link="${parent}" />
-        <child link="${prefix}gripper_base_link" />
+        <geometry><mesh filename="${mesh_url}${mesh_name}.STL" /></geometry>
+        <material name=""><color rgba="${color_rgba}" /></material>
+      </visual>
+      <collision>
+        <origin xyz="0 0 0" rpy="0 0 0" />
+        <geometry><mesh filename="${mesh_url}${mesh_name}.dae" /></geometry>
+      </collision>
+    </xacro:macro>
+    <!-- ========================================== -->
+    <!-- 4. ESTRUTURA MECÂNICA UNIFICADA            -->
+    <!-- ========================================== -->
+    <!-- Tool frame -->
+    <link name="${pfx}tool_frame"/>
+    <joint name="${pfx}tool_frame_joint" type="fixed">
+        <origin xyz="0 0 0.130" rpy="0 0 1.57079632679" />
+        <parent link="${prnt}" />
+        <child link="${pfx}tool_frame" />
         <axis xyz="0 0 0" />
-      </joint>
-      <link name="${prefix}gripper_base_link">
-        <inertial>
-          <origin xyz="4.03E-06 1.08E-05 0.041397" rpy="0 0 0" />
-          <mass value="0.1395" />
-          <inertia ixx="0.00011614" ixy="1E-08" ixz="4E-08" iyy="0.00010327" iyz="0" izz="9.707E-05" />
-        </inertial>
-        <visual>
-          <origin xyz="0 0 0" rpy="0 0 0" />
-          <geometry>
-            <mesh filename="file://$(find kortex_description)/grippers/gen3_lite_2f/meshes/gripper_base_link.STL" />
-          </geometry>
-          <material name="">
-            <color rgba="0.803 0.824 0.820 1" />
-          </material>
-        </visual>
-        <collision>
-          <origin xyz="0 0 0" rpy="0 0 0" />
-          <geometry>
-            <mesh filename="file://$(find kortex_description)/grippers/gen3_lite_2f/meshes/gripper_base_link.STL" />
-          </geometry>
-        </collision>
-      </link>
-      <gazebo reference="${prefix}gripper_base_link">
-        <material>Kortex/Gray</material>
-      </gazebo>
-      <link name="${prefix}right_finger_prox_link">
+    </joint>
+    <!-- Gripper Base -->
+    <joint name="${pfx}gripper_base_joint" type="fixed">
+      <origin xyz="0 0 0" rpy="0 0 0" />
+      <parent link="${prnt}" />
+      <child link="${pfx}gripper_base_link" />
+      <axis xyz="0 0 0" />
+    </joint>
+    <link name="${pfx}gripper_base_link">
+      <inertial>
+        <origin xyz="4.03E-06 1.08E-05 0.041397" rpy="0 0 0" />
+        <mass value="0.1395" />
+        <inertia ixx="0.00011614" ixy="1E-08" ixz="4E-08" iyy="0.00010327" iyz="0" izz="9.707E-05" />
+      </inertial>
+      <xacro:gripper_mesh mesh_name="gripper_base_link" color_rgba="0.803 0.824 0.820 1" />
+    </link>
+    <gazebo reference="${pfx}gripper_base_link"><material>Kortex/Gray</material></gazebo>
+    <!-- Right Finger Prox -->
+    <link name="${pfx}right_finger_prox_link">
       <inertial>
         <origin xyz="0.020257 0.0063483 6.991E-05" rpy="0 0 0" />
@@ -81,383 +125,17 @@
         <inertia ixx="2.29E-06" ixy="1.43E-06" ixz="0" iyy="4.56E-06" iyz="0" izz="4.77E-06" />
       </inertial>
-      <visual>
-        <origin xyz="0 0 0" rpy="0 0 0" />
-        <geometry>
-          <mesh filename="file://$(find kortex_description)/grippers/gen3_lite_2f/meshes/right_finger_prox_link.STL" />
-        </geometry>
-        <material name="">
-            <color rgba="0.803 0.824 0.820 1" />
-        </material>
-      </visual>
-      <collision>
-        <origin xyz="0 0 0" rpy="0 0 0" />
-        <geometry>
-          <mesh filename="file://$(find kortex_description)/grippers/gen3_lite_2f/meshes/right_finger_prox_link.STL" />
-        </geometry>
-      </collision>
-      </link>
-      <gazebo reference="${prefix}right_finger_prox_link">
-        <material>Kortex/Gray</material>
-      </gazebo>
-      <joint name="${prefix}right_finger_bottom_joint" type="revolute">
-        <origin xyz="0 -0.030501 0.070003" rpy="1.571 0.611 1.571" />
-        <parent link="${prefix}gripper_base_link" />
-        <child link="${prefix}right_finger_prox_link" />
-        <axis xyz="0 0 -1" />
-        <limit lower="-0.1" upper="0.96" effort="10" velocity="0.6" />
-        <dynamics damping="0.1" friction="1"/>
-      </joint>
-      <link name="${prefix}right_finger_dist_link">
-        <inertial>
-          <origin xyz="0.018488 0.0011091 0" rpy="0 0 0" />
-          <mass value="0.010748" />
-          <inertia ixx="6.3E-07" ixy="3.2E-07" ixz="0" iyy="1.83E-06" iyz="0" izz="1.61E-06" />
-        </inertial>
-        <visual>
-          <origin xyz="0 0 0" rpy="0 0 0" />
-          <geometry>
-            <mesh filename="file://$(find kortex_description)/grippers/gen3_lite_2f/meshes/right_finger_dist_link.STL" />
-          </geometry>
-          <material name="">
-            <color rgba="0 0.055 0.525 1" />
-          </material>
-        </visual>
-        <collision>
-          <origin xyz="0 0 0" rpy="0 0 0" />
-          <geometry>
-            <mesh filename="file://$(find kortex_description)/grippers/gen3_lite_2f/meshes/right_finger_dist_link.STL" />
-          </geometry>
-        </collision>
-      </link>
-      <gazebo reference="${prefix}right_finger_dist_link">
-        <material>Kortex/Blue</material>
-      </gazebo>
-      <joint name="${prefix}right_finger_tip_joint" type="revolute">
-        <origin xyz="-0.045636 0.020423 0" rpy="0 0 0" />
-        <parent link="${prefix}right_finger_prox_link" />
-        <child link="${prefix}right_finger_dist_link" />
-        <axis xyz="0 0 1" />
-        <limit lower="-0.50" upper="0.21" effort="1000" velocity="1000" /> <!--limit lower="-1.03" upper="0.21" effort="1000" velocity="1000" /-->
-        <mimic joint="${prefix}right_finger_bottom_joint" multiplier="-0.276" offset="-0.1" />
-      </joint>
-      <link name="${prefix}left_finger_prox_link">
-        <inertial>
-          <origin xyz="0.020257 0.0063483 6.99E-05" rpy="0 0 0" />
-          <mass value="0.018385" />
-          <inertia ixx="2.29E-06" ixy="1.43E-06" ixz="0" iyy="4.56E-06" iyz="0" izz="4.77E-06" />
-        </inertial>
-        <visual>
-          <origin xyz="0 0 0" rpy="0 0 0" />
-          <geometry>
-            <mesh filename="file://$(find kortex_description)/grippers/gen3_lite_2f/meshes/left_finger_prox_link.STL" />
-          </geometry>
-          <material name="">
-            <color rgba="0.803 0.824 0.820 1" />
-          </material>
-        </visual>
-        <collision>
-          <origin xyz="0 0 0" rpy="0 0 0" />
-          <geometry>
-            <mesh filename="file://$(find kortex_description)/grippers/gen3_lite_2f/meshes/left_finger_prox_link.STL" />
-          </geometry>
-        </collision>
-      </link>
-      <gazebo reference="${prefix}left_finger_prox_link">
-        <material>Kortex/Gray</material>
-      </gazebo>
-      <joint name="${prefix}left_finger_bottom_joint" type="revolute">
-        <origin xyz="0 0.0305 0.070003" rpy="-1.571 0.611 -1.571" />
-        <parent link="${prefix}gripper_base_link" />
-        <child link="${prefix}left_finger_prox_link" />
-        <axis xyz="0 0 1" />
-        <limit lower="-0.1" upper="0.96" effort="10" velocity="0.6" />
-        <dynamics damping="0.1" friction="1"/>
-        <mimic joint="${prefix}right_finger_bottom_joint" multiplier="1.0" offset="0.0" />
-      </joint>
-      <link name="${prefix}left_finger_dist_link">
-        <inertial>
-          <origin xyz="-0.018488 0.0011091 0" rpy="0 0 0" />
-          <mass value="0.010748" />
-          <inertia ixx="6.3E-07" ixy="3.2E-07" ixz="0" iyy="1.83E-06" iyz="0" izz="1.61E-06" />
-        </inertial>
-        <visual>
-          <origin xyz="0 0 0" rpy="0 0 0" />
-          <geometry>
-            <mesh filename="file://$(find kortex_description)/grippers/gen3_lite_2f/meshes/left_finger_dist_link.STL" />
-          </geometry>
-          <material name="">
-            <color rgba="0 0.055 0.525 1" />
-          </material>
-        </visual>
-        <collision>
-          <origin xyz="0 0 0" rpy="0 0 0" />
-          <geometry>
-            <mesh filename="file://$(find kortex_description)/grippers/gen3_lite_2f/meshes/left_finger_dist_link.STL" />
-          </geometry>
-        </collision>
-      </link>
-      <gazebo reference="${prefix}left_finger_dist_link">
-        <material>Kortex/Blue</material>
-      </gazebo>
-      <joint name="${prefix}left_finger_tip_joint" type="revolute">
-        <origin xyz="-0.045636 -0.020423 6.9901E-05" rpy="0 0 0" />
-        <parent link="${prefix}left_finger_prox_link" />
-        <child link="${prefix}left_finger_dist_link" />
-        <axis xyz="0 0 -1" />
-        <limit lower="-0.50" upper="0.21" effort="1000" velocity="1000" /> <!--limit lower="-1.03" upper="0.21" effort="1000" velocity="1000" /-->
-        <mimic joint="${prefix}right_finger_bottom_joint" multiplier="-0.276" offset="-0.1" />
-      </joint>
-    </xacro:unless>
-  </xacro:if>
-  <xacro:unless value="${use_fake_hardware or sim_isaac or sim_gazebo}">
-    <xacro:unless value="${moveit_active}">
-        <!-- Tool frame used by the arm -->
-      <link name="${prefix}tool_frame"/>
-      <joint name="${prefix}tool_frame_joint" type="fixed">
-          <origin xyz="0 0 0.130" rpy="0 0 1.57079632679" />
-          <parent link="${parent}" />
-          <child link="${prefix}tool_frame" />
-          <axis xyz="0 0 0" />
-      </joint>
-      <!-- Gripper description -->
-      <joint name="${prefix}gripper_base_joint" type="fixed">
-        <origin xyz="0 0 0" rpy="0 0 0" />
-        <parent link="${parent}" />
-        <child link="${prefix}gripper_base_link" />
-        <axis xyz="0 0 0" />
-      </joint>
-      <link name="${prefix}gripper_base_link">
-        <inertial>
-          <origin xyz="4.03E-06 1.08E-05 0.041397" rpy="0 0 0" />
-          <mass value="0.1395" />
-          <inertia ixx="0.00011614" ixy="1E-08" ixz="4E-08" iyy="0.00010327" iyz="0" izz="9.707E-05" />
-        </inertial>
-        <visual>
-          <origin xyz="0 0 0" rpy="0 0 0" />
-          <geometry>
-            <mesh filename="file://$(find kortex_description)/grippers/gen3_lite_2f/meshes/gripper_base_link.STL" />
-          </geometry>
-          <material name="">
-            <color rgba="0.803 0.824 0.820 1" />
-          </material>
-        </visual>
-        <collision>
-          <origin xyz="0 0 0" rpy="0 0 0" />
-          <geometry>
-            <mesh filename="file://$(find kortex_description)/grippers/gen3_lite_2f/meshes/gripper_base_link.STL" />
-          </geometry>
-        </collision>
-      </link>
-      <gazebo reference="${prefix}gripper_base_link">
-        <material>Kortex/Gray</material>
-      </gazebo>
-      <link name="${prefix}right_finger_prox_link">
-      <inertial>
-        <origin xyz="0.020257 0.0063483 6.991E-05" rpy="0 0 0" />
-        <mass value="0.018385" />
-        <inertia ixx="2.29E-06" ixy="1.43E-06" ixz="0" iyy="4.56E-06" iyz="0" izz="4.77E-06" />
-      </inertial>
-      <visual>
-        <origin xyz="0 0 0" rpy="0 0 0" />
-        <geometry>
-          <mesh filename="file://$(find kortex_description)/grippers/gen3_lite_2f/meshes/right_finger_prox_link.STL" />
-        </geometry>
-        <material name="">
-            <color rgba="0.803 0.824 0.820 1" />
-        </material>
-      </visual>
-      <collision>
-        <origin xyz="0 0 0" rpy="0 0 0" />
-        <geometry>
-          <mesh filename="file://$(find kortex_description)/grippers/gen3_lite_2f/meshes/right_finger_prox_link.STL" />
-        </geometry>
-      </collision>
-      </link>
-      <gazebo reference="${prefix}right_finger_prox_link">
-        <material>Kortex/Gray</material>
-      </gazebo>
-      <!-- TODO(MarqRazz) look into why the joint and limits needed to be flipped and modified -->
-      <joint name="${prefix}right_finger_bottom_joint" type="revolute">
-        <origin xyz="0 -0.030501 0.070003" rpy="1.571 0.611 1.571" />
-        <parent link="${prefix}gripper_base_link" />
-        <child link="${prefix}right_finger_prox_link" />
-        <axis xyz="0 0 -1" />
-        <limit lower="0.0" upper="0.85" effort="50" velocity="0.6" />
-      </joint>
-      <link name="${prefix}right_finger_dist_link">
-        <inertial>
-          <origin xyz="0.018488 0.0011091 0" rpy="0 0 0" />
-          <mass value="0.010748" />
-          <inertia ixx="6.3E-07" ixy="3.2E-07" ixz="0" iyy="1.83E-06" iyz="0" izz="1.61E-06" />
-        </inertial>
-        <visual>
-          <origin xyz="0 0 0" rpy="0 0 0" />
-          <geometry>
-            <mesh filename="file://$(find kortex_description)/grippers/gen3_lite_2f/meshes/right_finger_dist_link.STL" />
-          </geometry>
-          <material name="">
-            <color rgba="0 0.055 0.525 1" />
-          </material>
-        </visual>
-        <collision>
-          <origin xyz="0 0 0" rpy="0 0 0" />
-          <geometry>
-            <mesh filename="file://$(find kortex_description)/grippers/gen3_lite_2f/meshes/right_finger_dist_link.STL" />
-          </geometry>
-        </collision>
-      </link>
-      <gazebo reference="${prefix}right_finger_dist_link">
-        <material>Kortex/Blue</material>
-      </gazebo>
-      <joint name="${prefix}right_finger_tip_joint" type="revolute">
-        <origin xyz="-0.045636 0.020423 0" rpy="0 0 0" />
-        <parent link="${prefix}right_finger_prox_link" />
-        <child link="${prefix}right_finger_dist_link" />
-        <axis xyz="0 0 1" />
-        <limit lower="-0.50" upper="0.21" effort="1000" velocity="1000" /> <!--limit lower="-1.03" upper="0.21" effort="1000" velocity="1000" /-->
-        <mimic joint="${prefix}right_finger_bottom_joint" multiplier="-0.276" offset="-0.1" />
-      </joint>
-      <link name="${prefix}left_finger_prox_link">
-        <inertial>
-          <origin xyz="0.020257 0.0063483 6.99E-05" rpy="0 0 0" />
-          <mass value="0.018385" />
-          <inertia ixx="2.29E-06" ixy="1.43E-06" ixz="0" iyy="4.56E-06" iyz="0" izz="4.77E-06" />
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